Commit message: Add ur_description

File: hrwros_week2/hrwros/hrwros_support/urdf/hrwros.xacro (robot description, xacro)
@@ -12,6 +12,9 @@
   </xacro:robot_pedestal_urdf>
   <!-- Robot1 -->
-  <xacro:include filename="$(find ur_description)/urdf/ur10.urdf.xacro"/>
-  <xacro:ur10_robot prefix="robot1_" joint_limited="true"/>
+  <xacro:include filename="$(find hrwros_support)/urdf/arm_robot/arm_robot_prop.urdf.xacro"/>
+  <xacro:include filename="$(find hrwros_support)/urdf/arm_robot/arm_robot.urdf.xacro"/>
+  <xacro:custom_arm_robot name="robot1" ur_type="ur10" parent="robot1_pedestal_link">
+    <origin xyz="0 0 0.95" rpy="0 0 0" />
+  </xacro:custom_arm_robot>
   <!-- Vacuum Gripper1 -->
   <xacro:include filename="$(find hrwros_support)/urdf/vacuum_gripper/vacuum_gripper.urdf.xacro"/>
@@ -29,4 +32,5 @@
     <child link="world_interface" />
   </joint>
+  <!-- #### -->
   <!-- robot1-pedestal to world. -->
   <joint name="robot1_pedestal_to_world_interface" type="fixed">
@@ -34,10 +38,4 @@
     <child link="robot1_pedestal_link" />
     <origin xyz="0.5 1.8 0.0" rpy="0.0 0.0 0.0"/>
-  </joint>
-  <!-- robot1 to pedestal. -->
-  <joint name="robot1_to_pedestal" type="fixed">
-  <origin xyz="0 0 0.95" rpy="0 0 0" />
-  <parent link="robot1_pedestal_link" />
-  <child link="robot1_base_link" />
   </joint>
   <!-- gripper1 to robot1. -->
