Commit message: fix hrwros.xacro

File: hrwros_week2/hrwros/hrwros_support/urdf/arm_robot/arm_robot.urdf.xacro (robot description, xacro)
@@ -68,4 +68,7 @@
         </gazebo>
     </xacro:if>
+  <!-- Vacuum Gripper1 -->
+  <xacro:include filename="$(find hrwros_support)/urdf/vacuum_gripper/vacuum_gripper.urdf.xacro"/>
+  <xacro:vacuum_gripper_urdf prefix="${name}" parent="${name}_tool0"/>
     </xacro:macro>
 </robot>

File: hrwros_week2/hrwros/hrwros_support/urdf/hrwros.xacro (robot description, xacro)
@@ -17,7 +17,4 @@
     <origin xyz="0 0 0.95" rpy="0 0 0" />
   </xacro:custom_arm_robot>
-  <!-- Vacuum Gripper1 -->
-  <xacro:include filename="$(find hrwros_support)/urdf/vacuum_gripper/vacuum_gripper.urdf.xacro"/>
-  <xacro:vacuum_gripper_urdf prefix="vacuum_gripper1" parent="robot1_tool0" robot_name="robot1"/>
   <!-- bins -->
   <xacro:include filename="$(find hrwros_support)/urdf/bin/bin.urdf.xacro"/>

File: hrwros_week2/hrwros/hrwros_support/urdf/vacuum_gripper/vacuum_gripper.urdf.xacro (robot description, xacro)
@@ -1,7 +1,7 @@
 <?xml version="1.0"?>
 <robot xmlns:xacro="http://www.ros.org/wiki/xacro">
-  <xacro:macro name="vacuum_gripper_urdf" params="prefix parent robot_name">
+  <xacro:macro name="vacuum_gripper_urdf" params="prefix parent">
     <!-- link list -->
-    <link name="${prefix}_base_link">
+    <link name="${prefix}_vacuum_gripper_base_link" >
       <visual>
         <origin xyz="0 0 0" rpy="0 0 0" />
@@ -28,5 +28,5 @@
       </inertial>
     </link>
-    <link name="${prefix}_suction_cup">
+    <link name="${prefix}_vacuum_gripper_suction_cup">
       <visual>
         <origin xyz="0 0 0" rpy="0 0 0" />
@@ -54,13 +54,13 @@
     </link>
     <!-- joint list -->
-    <joint name="${prefix}_joint" type="fixed">
+  <joint name="${prefix}_to_vacuum_gripper_joint_1" type="fixed">
+    <parent link="${parent}" />
+    <child link="${prefix}_vacuum_gripper_base_link" />
+  </joint>
+    <joint name="${prefix}_to_vacuum_gripper_joint_2" type="fixed">
       <origin xyz="0 0 0.01" rpy="0 0 0" />
-      <parent link="${prefix}_base_link" />
-      <child link="${prefix}_suction_cup" />
+      <parent link="${prefix}_vacuum_gripper_base_link"  />
+      <child link="${prefix}_vacuum_gripper_suction_cup" />
     </joint>
-  <joint name="{prefix}_to_${robot_name}" type="fixed">
-    <parent link="${parent}" />
-    <child link="${prefix}_base_link" />
-  </joint>
   </xacro:macro>
 </robot>
