Commit message: fix hrwros.xacro

File: hrwros_week2/hrwros/hrwros_support/urdf/bin/bin.urdf.xacro (robot description, xacro)
@@ -1,7 +1,7 @@
 <?xml version="1.0"?>
 <robot xmlns:xacro="http://www.ros.org/wiki/xacro">
-  <xacro:macro name="bin_urdf" params="prefix">
+  <xacro:macro name="bin_urdf" params="prefix parent">
     <!-- link list -->
-    <link name="${prefix}base_link">
+    <link name="${prefix}_base_link">
       <visual>
         <origin xyz="0 0 0" rpy="0 0 0" />
@@ -24,24 +24,25 @@
       <inertial>
         <origin xyz="0 0 0" rpy="0 0 0" />
-        <inertia ixx="1.0" ixy="0" ixz="0"
-                 iyy="1.0" iyz="0"
-                 izz="1.0" />
+        <inertia ixx="1.0" ixy="0" ixz="0" iyy="1.0" iyz="0" izz="1.0" />
         <mass value="100" />
       </inertial>
     </link>
-    <link name="${prefix}drop_point">
+    <link name="${prefix}_drop_point">
       <inertial>
         <origin xyz="0 0 0" rpy="0 0 0" />
-        <inertia ixx="1.0" ixy="0" ixz="0"
-                 iyy="1.0" iyz="0"
-                 izz="1.0" />
+        <inertia ixx="1.0" ixy="0" ixz="0" iyy="1.0" iyz="0" izz="1.0" />
         <mass value="1.0" />
       </inertial>
     </link>
     <!-- joint list -->
-    <joint name="${prefix}joint_1" type="fixed">
+    <joint name="${prefix}_joint_1" type="fixed">
+      <parent link="${parent}" />
+      <child link="${prefix}_base_link" />
+      <origin xyz="-0.3 1.2 0.0" rpy="0 0 0" />
+    </joint>
+    <joint name="${prefix}_joint_2" type="fixed">
       <origin xyz="0 0 1.0" rpy="0 0 0" />
-      <parent link="${prefix}base_link" />
-      <child link="${prefix}drop_point" />
+      <parent link="${prefix}_base_link" />
+      <child link="${prefix}_drop_point" />
     </joint>
   </xacro:macro>

File: hrwros_week2/hrwros/hrwros_support/urdf/hrwros.xacro (robot description, xacro)
@@ -5,8 +5,8 @@
   <!-- workcell -->
   <xacro:include filename="$(find hrwros_support)/urdf/workcell/workcell.urdf.xacro"/>
-  <xacro:workcell_urdf workcell_parent="world_interface"/>
+  <xacro:workcell_urdf parent="world"/>
   <!-- Robot1 Pedestal -->
   <xacro:include filename="$(find hrwros_support)/urdf/robot_pedestal/robot_pedestal.urdf.xacro"/>
-  <xacro:robot_pedestal_urdf pedestal_prefix="robot1_" pedestal_parent="world_interface" pedestal_height="0.95">
+  <xacro:robot_pedestal_urdf prefix="robot1" parent="world" pedestal_height="0.95">
     <origin xyz="0.5 1.8 0.0" rpy="0 0 0"/>
   </xacro:robot_pedestal_urdf>
@@ -19,58 +19,7 @@
   <!-- Vacuum Gripper1 -->
   <xacro:include filename="$(find hrwros_support)/urdf/vacuum_gripper/vacuum_gripper.urdf.xacro"/>
-  <xacro:vacuum_gripper_urdf prefix="vacuum_gripper1_" joint_prefix="vacuum_gripper1_joint"/>
+  <xacro:vacuum_gripper_urdf prefix="vacuum_gripper1" parent="robot1_tool0" robot_name="robot1"/>
   <!-- bins -->
   <xacro:include filename="$(find hrwros_support)/urdf/bin/bin.urdf.xacro"/>
-  <xacro:bin_urdf prefix="bin_1_"/>
-  <xacro:bin_urdf prefix="bin_2_"/>
-  <xacro:bin_urdf prefix="bin_3_"/>
-  <xacro:bin_urdf prefix="bin_4_"/>
-  <xacro:bin_urdf prefix="bin_5_"/>
-  <!-- Joints -->
-  <joint name="world_interface_to_world" type="fixed">
-    <parent link="world" />
-    <child link="world_interface" />
-  </joint>
-  <!-- #### -->
-  <!-- robot1-pedestal to world. -->
-  <joint name="robot1_pedestal_to_world_interface" type="fixed">
-    <parent link="world_interface" />
-    <child link="robot1_pedestal_link" />
-    <origin xyz="0.5 1.8 0.0" rpy="0.0 0.0 0.0"/>
-  </joint>
-  <!-- gripper1 to robot1. -->
-  <joint name="gripper1_to_robot1" type="fixed">
-    <parent link="robot1_tool0" />
-    <child link="vacuum_gripper1_base_link" />
-  </joint>
-  <!-- bin 1 -->
-  <joint name="bin_1_joint" type="fixed">
-    <parent link="world_interface" />
-    <child link="bin_1_base_link" />
-    <origin xyz="-0.3 1.2 0.0" rpy="0 0 0" />
-  </joint>
-  <!-- bin 2 -->
-  <joint name="bin_2_joint" type="fixed">
-    <parent link="world_interface" />
-    <child link="bin_2_base_link" />
-    <origin xyz="-0.3 0.4 0.0" rpy="0 0 0" />
-  </joint>
-  <!-- bin 3 -->
-  <joint name="bin_3_joint" type="fixed">
-    <parent link="world_interface" />
-    <child link="bin_3_base_link" />
-    <origin xyz="-0.3 -0.4 0.0" rpy="0 0 0" />
-  </joint>
-  <!-- bin 4 -->
-  <joint name="bin_4_joint" type="fixed">
-    <parent link="world_interface" />
-    <child link="bin_4_base_link" />
-    <origin xyz="-0.3 -1.2 0.0" rpy="0 0 0" />
-  </joint>
-  <!-- bin 5 -->
-  <joint name="bin_5_joint" type="fixed">
-    <parent link="world_interface" />
-    <child link="bin_5_base_link" />
-    <origin xyz="-0.3 -2.0 0.0" rpy="0 0 0" />
-  </joint>
+  <xacro:bin_urdf prefix="bin_1" parent="world"/>
 </robot>

File: hrwros_week2/hrwros/hrwros_support/urdf/robot_pedestal/robot_pedestal.urdf.xacro (robot description, xacro)
@@ -2,11 +2,6 @@
 <robot name="robot_pedestal_urdf" xmlns:xacro="http://www.ros.org/wiki/xacro">
 <!-- robot pedestal -->
-<xacro:macro name = "robot_pedestal_urdf" params = "pedestal_prefix pedestal_parent pedestal_height *origin">
-  <joint name="${pedestal_prefix}pedestal_joint" type="fixed">
-    <xacro:insert_block name="origin" />
-    <parent link="${pedestal_parent}"/>
-    <child link="${pedestal_prefix}pedestal_link"/>
-  </joint>
-  <link name="${pedestal_prefix}pedestal_link">
+<xacro:macro name = "robot_pedestal_urdf" params = "prefix parent pedestal_height *origin">
+  <link name="${prefix}_pedestal_link">
     <visual>
       <origin xyz="0 0 ${0.5*pedestal_height}"/>
@@ -30,5 +25,10 @@
     </inertial>
   </link>
-  <gazebo reference="${pedestal_prefix}pedestal_link">
+  <joint name="${prefix}_pedestal_joint" type="fixed">
+    <xacro:insert_block name="origin" />
+    <parent link="${parent}"/>
+    <child link="${prefix}_pedestal_link"/>
+  </joint>
+  <gazebo reference="${prefix}_pedestal_link">
     <material>Gazebo/Blue</material>
   </gazebo>

File: hrwros_week2/hrwros/hrwros_support/urdf/vacuum_gripper/vacuum_gripper.urdf.xacro (robot description, xacro)
@@ -1,7 +1,7 @@
 <?xml version="1.0"?>
 <robot xmlns:xacro="http://www.ros.org/wiki/xacro">
-  <xacro:macro name="vacuum_gripper_urdf" params="prefix joint_prefix">
+  <xacro:macro name="vacuum_gripper_urdf" params="prefix parent robot_name">
     <!-- link list -->
-    <link name="${prefix}base_link">
+    <link name="${prefix}_base_link">
       <visual>
         <origin xyz="0 0 0" rpy="0 0 0" />
@@ -28,5 +28,5 @@
       </inertial>
     </link>
-    <link name="${prefix}suction_cup">
+    <link name="${prefix}_suction_cup">
       <visual>
         <origin xyz="0 0 0" rpy="0 0 0" />
@@ -54,9 +54,13 @@
     </link>
     <!-- joint list -->
-    <joint name="${joint_prefix}" type="fixed">
+    <joint name="${prefix}_joint" type="fixed">
       <origin xyz="0 0 0.01" rpy="0 0 0" />
-      <parent link="${prefix}base_link" />
-      <child link="${prefix}suction_cup" />
+      <parent link="${prefix}_base_link" />
+      <child link="${prefix}_suction_cup" />
     </joint>
+  <joint name="{prefix}_to_${robot_name}" type="fixed">
+    <parent link="${parent}" />
+    <child link="${prefix}_base_link" />
+  </joint>
   </xacro:macro>
 </robot>

File: hrwros_week2/hrwros/hrwros_support/urdf/workcell/workcell.urdf.xacro (robot description, xacro)
@@ -1,7 +1,6 @@
 <?xml version="1.0" ?>
 <robot name="workcell_urdf" xmlns:xacro="http://www.ros.org/wiki/xacro">
-    <xacro:macro name="workcell_urdf" params="workcell_parent">
+    <xacro:macro name="workcell_urdf" params="parent">
     <!-- Links -->
-    <link name="world_interface"/>
     <link name="workcell">
       <visual>
@@ -22,6 +21,6 @@
       </inertial>
     </link>
-    <joint name="workcell_to_world_interface" type="fixed">
-      <parent link="${workcell_parent}" />
+    <joint name="workcell_to_${parent}" type="fixed">
+      <parent link="${parent}" />
       <child link="workcell" />
       <origin xyz="0 0 0" rpy="0 0 ${radians(90)}" />

Commit message: Add the arm robots

File: hrwros_week2/hrwros/hrwros_support/urdf/bin/bin.urdf.xacro (robot description, xacro)
@@ -1,5 +1,5 @@
 <?xml version="1.0"?>
 <robot xmlns:xacro="http://www.ros.org/wiki/xacro">
-  <xacro:macro name="bin_urdf" params="prefix parent">
+  <xacro:macro name="bin_urdf" params="prefix parent *origin">
     <!-- link list -->
     <link name="${prefix}_base_link">
@@ -39,5 +39,5 @@
       <parent link="${parent}" />
       <child link="${prefix}_base_link" />
-      <origin xyz="-0.3 1.2 0.0" rpy="0 0 0" />
+      <xacro:insert_block name="origin" />
     </joint>
     <joint name="${prefix}_joint_2" type="fixed">

File: hrwros_week2/hrwros/hrwros_support/urdf/hrwros.xacro (robot description, xacro)
@@ -1,4 +1,5 @@
 <?xml version="1.0" ?>
-<robot name="robot" xmlns:xacro="http://www.ros.org/wiki/xacro">
+<robot name="robot"
+  xmlns:xacro="http://www.ros.org/wiki/xacro">
   <!-- world -->
   <link name="world" />
@@ -6,17 +7,18 @@
   <xacro:include filename="$(find hrwros_support)/urdf/workcell/workcell.urdf.xacro"/>
   <xacro:workcell_urdf parent="world"/>
-  <!-- Robot1 Pedestal -->
-  <xacro:include filename="$(find hrwros_support)/urdf/robot_pedestal/robot_pedestal.urdf.xacro"/>
-  <xacro:robot_pedestal_urdf prefix="robot1" parent="world" pedestal_height="0.95">
+  <!-- Robots -->
+  <xacro:include filename="$(find hrwros_support)/urdf/container_arm_robot_pedestal/container_arm_robot_pedestal.urdf.xacro"/>
+  <!-- Robot1 -->
+  <xacro:container_arm_robot_pedestal_urdf robot_name="robot1" ur_type="ur10" parent_pedestal="world" height_pedestal="0.95">
     <origin xyz="0.5 1.8 0.0" rpy="0 0 0"/>
-  </xacro:robot_pedestal_urdf>
-  <!-- Robot1 -->
-  <xacro:include filename="$(find hrwros_support)/urdf/arm_robot/arm_robot_prop.urdf.xacro"/>
-  <xacro:include filename="$(find hrwros_support)/urdf/arm_robot/arm_robot.urdf.xacro"/>
-  <xacro:custom_arm_robot name="robot1" ur_type="ur10" parent="robot1_pedestal_link">
-    <origin xyz="0 0 0.95" rpy="0 0 0" />
-  </xacro:custom_arm_robot>
-  <!-- bins -->
+  </xacro:container_arm_robot_pedestal_urdf>
+  <!-- Robot2 -->
+  <xacro:container_arm_robot_pedestal_urdf robot_name="robot2" ur_type="ur10" parent_pedestal="world" height_pedestal="0.5">
+    <origin xyz="-7.6 -0.5 0.0" rpy="0 0 0"/>
+  </xacro:container_arm_robot_pedestal_urdf>
+  <!-- bin1 -->
   <xacro:include filename="$(find hrwros_support)/urdf/bin/bin.urdf.xacro"/>
-  <xacro:bin_urdf prefix="bin_1" parent="world"/>
+  <xacro:bin_urdf prefix="bin_1" parent="world">
+    <origin xyz="-7.6 -1.7 0" rpy="0 0 0" />
+  </xacro:bin_urdf>
 </robot>
