Commit message: Add hrwros_assignment1.xacro

File: hrwros_week2/hrwros_assignments/hrwros_week2_assignment/urdf/hrwros_assignment1.xacro (robot description, xacro)
@@ -21,4 +21,8 @@
     <origin xyz="-8.0 -2.2 0" rpy="0 0 0" />
   </xacro:bin_urdf>
+  <!-- bin2 -->
+  <xacro:bin_urdf prefix="bin_2" parent="world">
+    <origin xyz="2.5 -3.2 0" rpy="0 0 0" />
+  </xacro:bin_urdf>
   <!-- Add your solution to assignment 1 here -->
 </robot>
