Commit message: Add hrwros_assignment1.xacro

File: hrwros_week2/hrwros_assignments/hrwros_week2_assignment/urdf/hrwros_assignment2.xacro (robot description, xacro)
@@ -22,3 +22,8 @@
   </xacro:bin_urdf>
   <!-- Add your solution to assignment 2 here -->
+  <!-- sphere1 -->
+  <xacro:include filename="$(find hrwros_week2_assignment)/urdf/include/sphere.xacro"/>
+  <xacro:sphere_urdf prefix="sphere_1" parent="world" radius="0.4">
+    <origin xyz="5.2 -6 0" rpy="0 0 0" />
+  </xacro:sphere_urdf>
 </robot>
