Commit message: Add hrwros_assignment3.xacro

File: hrwros_week2/hrwros_assignments/hrwros_week2_assignment/urdf/hrwros_assignment3.xacro (robot description, xacro)
@@ -12,8 +12,4 @@
     <origin xyz="0.5 1.8 0.0" rpy="0 0 0"/>
   </xacro:container_arm_robot_pedestal_urdf>
-  <!-- Robot2 -->
-  <xacro:container_arm_robot_pedestal_urdf robot_name="robot2" ur_type="ur5" parent_pedestal="world" height_pedestal="0.6">
-    <origin xyz="-7.8 -1.5 0" rpy="0 0 0"/>
-  </xacro:container_arm_robot_pedestal_urdf>
   <!-- bin1 -->
   <xacro:include filename="$(find hrwros_support)/urdf/bin/bin.urdf.xacro"/>
@@ -22,3 +18,8 @@
   </xacro:bin_urdf>
   <!-- Add your solution to assignment 3 here -->
+  <xacro:include filename="$(find hrwros_week2_assignment)/urdf/include/lrmate200ic_pedestal_urdf.xacro"/>
+  <!-- Robot2 -->
+  <xacro:lrmate200ic_pedestal_urdf robot_name="robot2"  parent_pedestal="world" height_pedestal="0.6">
+    <origin xyz="-7.8 -1.5 0" rpy="0 0 0"/>
+  </xacro:lrmate200ic_pedestal_urdf>
 </robot>
