Commit message: fix

File: hrwros_week3/hrwros_support/urdf/workcell/workcell.xacro (robot description, xacro)
@@ -1,5 +1,7 @@
 <?xml version="1.0" ?>
-<robot name="workcell" xmlns:xacro="http://www.ros.org/wiki/xacro">
-  <xacro:arg name="workcell_parent_name" default="world"/>
+<robot name="workcell"
+  xmlns:xacro="http://www.ros.org/wiki/xacro">
+  <link name="world_interface" />
+  <xacro:arg name="workcell_parent_name" default="world_interface"/>
   <!-- URDF -->
   <xacro:include filename="$(find hrwros_support)/urdf/workcell/workcell.urdf.xacro"/>
