Commit message: fix

File: hrwros_week3/hrwros_support/urdf/workcell/workcell.urdf.xacro (robot description, xacro)
@@ -3,4 +3,5 @@
     <xacro:macro name="workcell_urdf" params="workcell_parent_name">
     <!-- Links -->
+    <link name="world_interface"/>
     <link name="workcell">
       <visual>

File: hrwros_week3/hrwros_support/urdf/workcell/workcell.xacro (robot description, xacro)
@@ -2,5 +2,4 @@
 <robot name="workcell"
   xmlns:xacro="http://www.ros.org/wiki/xacro">
-  <link name="world_interface" />
   <xacro:arg name="workcell_parent_name" default="world_interface"/>
   <!-- URDF -->

Commit message: change collision workcell for navigation purpose

File: hrwros_week3/hrwros_support/urdf/workcell/workcell.urdf.xacro (robot description, xacro)
@@ -11,5 +11,6 @@
       <collision>
         <geometry>
-          <mesh filename="file://$(find hrwros_support)/meshes/workcell/collision/workcell.dae"/>
+          <!-- <mesh filename="file://$(find hrwros_support)/meshes/workcell/collision/workcell.dae"/> -->
+          <mesh filename="file://$(find hrwros_support)/meshes/workcell/visual/workcell.dae"/>"/>
         </geometry>
       </collision>
