Commit message: Modify hrwros.xacro

File: hrwros_week3/hrwros_support/urdf/break_beam/break_beam.urdf.xacro (robot description, xacro)
@@ -1,5 +1,6 @@
 <?xml version="1.0"?>
-<robot name="break_beam_urdf" xmlns:xacro="http://www.ros.org/wiki/xacro">
-  <xacro:macro name="break_beam_urdf" params="prefix parent">
+<robot name="break_beam_urdf"
+  xmlns:xacro="http://www.ros.org/wiki/xacro">
+  <xacro:macro name="break_beam_urdf" params="prefix parent *origin">
     <!-- link list -->
     <link name="${prefix}${parent}"/>
@@ -23,16 +24,19 @@
       <inertial>
         <origin xyz="0 0 0" rpy="0 0 0" />
-        <inertia ixx="0.1" ixy="0" ixz="0"
-                 iyy="0.1" iyz="0"
-                 izz="0.1" />
+        <inertia ixx="0.1" ixy="0" ixz="0" iyy="0.1" iyz="0" izz="0.1" />
         <mass value="1" />
       </inertial>
     </link>
     <link name="${prefix}optical_link"/>
+    <!-- external parent joint -->
+    <joint name="${prefix}break_beam_joint" type="fixed">
+      <parent link="${parent}" />
+      <child link="${prefix}${parent}" />
+    </joint>
     <!-- joint list -->
     <joint name="${prefix}world_joint" type="fixed">
       <parent link="${prefix}${parent}" />
       <child link="${prefix}base_link" />
-      <origin xyz="1.6 1.9 0.925" rpy="0 0 ${radians(180)}" />
+      <xacro:insert_block name="origin" />
     </joint>
     <joint name="${prefix}joint_1" type="fixed">
@@ -41,9 +45,4 @@
       <origin xyz="0.025 0 0" rpy="0 0 0" />
     </joint>
-    <!-- external parent joint -->
-    <joint name="${prefix}break_beam_joint" type="fixed">
-      <parent link="${parent}" />
-      <child link="${prefix}${parent}" />
-    </joint>
   </xacro:macro>
 </robot>

File: hrwros_week3/hrwros_support/urdf/hrwros.xacro (robot description, xacro)
@@ -35,4 +35,6 @@
   </xacro:logical_camera_urdf>
   <!-- Break Beam -->
-  <xacro:break_beam_urdf prefix="break_beam_" parent="world"/>
+  <xacro:break_beam_urdf prefix="break_beam_" parent="world">
+    <origin xyz="1.6 1.9 0.925" rpy="0 0 ${radians(180)}" />
+  </xacro:break_beam_urdf>
 </robot>

Commit message: fix

File: hrwros_week3/hrwros_support/urdf/break_beam/break_beam.urdf.xacro (robot description, xacro)
@@ -4,5 +4,5 @@
   <xacro:macro name="break_beam_urdf" params="prefix *origin">
     <!-- link list -->
-    <link name="${prefix}world"/>
+    <link name="${prefix}world_interface"/>
     <link name="${prefix}base_link">
       <visual>
@@ -30,10 +30,6 @@
     <link name="${prefix}optical_link"/>
     <!-- joint list -->
-    <joint name="${prefix}joint" type="fixed">
-      <parent link="world" />
-      <child link="${prefix}world" />
-    </joint>
     <joint name="${prefix}world_joint" type="fixed">
-      <parent link="${prefix}world" />
+      <parent link="${prefix}world_interface" />
       <child link="${prefix}base_link" />
       <xacro:insert_block name="origin" />

File: hrwros_week3/hrwros_support/urdf/hrwros.xacro (robot description, xacro)
@@ -22,8 +22,8 @@
   <xacro:arg name="vacuum_gripper2" default="vacuum_gripper2_"/>
   <!-- Workcell -->
-  <xacro:workcell_urdf workcell_parent_name="world"/>
+  <xacro:workcell_urdf workcell_parent_name="world_interface"/>
   <!-- Robots -->
   <!-- Robot1 Pedestal -->
-  <xacro:robot_pedestal_urdf pedestal_prefix="$(arg robot1)_" pedestal_parent="world" pedestal_height="$(arg pedestal1_height)">
+  <xacro:robot_pedestal_urdf pedestal_prefix="$(arg robot1)_" pedestal_parent="world_interface" pedestal_height="$(arg pedestal1_height)">
     <origin xyz="0.5 1.8 0.0" rpy="0 0 0"/>
   </xacro:robot_pedestal_urdf>
@@ -35,5 +35,5 @@
   <xacro:vacuum_gripper_urdf prefix="$(arg vacuum_gripper1)" />
   <!-- Robot2 Pedestal -->
-  <xacro:robot_pedestal_urdf pedestal_prefix="$(arg robot2)_" pedestal_parent="world" pedestal_height="$(arg pedestal2_height)">
+  <xacro:robot_pedestal_urdf pedestal_prefix="$(arg robot2)_" pedestal_parent="world_interface" pedestal_height="$(arg pedestal2_height)">
     <origin xyz="-7.8 -1.5 0.0" rpy="0 0 0"/>
   </xacro:robot_pedestal_urdf>
@@ -63,4 +63,8 @@
   </xacro:break_beam_urdf>
   <!-- Joints -->
+ <joint name="world_interface_to_world" type="fixed">
+    <parent link="world" />
+    <child link="world_interface" />
+  </joint>
   <!-- gripper1 to robot1. -->
   <joint name="gripper1_to_robot1" type="fixed">
@@ -73,3 +77,8 @@
     <child link="$(arg vacuum_gripper2)base_link" />
   </joint>
+  <!-- break beam to world. -->
+  <joint name="break_beam_joint" type="fixed">
+    <parent link="world_interface" />
+    <child link="break_beam_world_interface" />
+  </joint>
 </robot>
