Commit message: Fix

File: hrwros_week3/hrwros_support/urdf/logical_camera/logical_camera.urdf.xacro (robot description, xacro)
@@ -7,5 +7,5 @@
     <joint name="${prefix}logical_camera_joint" type="fixed">
 	<xacro:insert_block name="origin" />
-	<parent link="world"/>
+	<parent link="world_interface"/>
 	<child link="${prefix}base_link"/>
     </joint>

File: hrwros_week3/hrwros_support/urdf/robot_pedestal/robot1_pedestal.xacro (robot description, xacro)
@@ -2,5 +2,5 @@
 <robot name="robot_pedestal" xmlns:xacro="http://www.ros.org/wiki/xacro">
   <xacro:arg name="pedestal_prefix" default="robot1"/>
-  <xacro:arg name="pedestal_parent" default="world"/>
+  <xacro:arg name="pedestal_parent" default="world_interface"/>
   <xacro:arg name="pedestal_height" default="0.95"/>
   <link name="world_interface"/>

File: hrwros_week3/hrwros_support/urdf/robot_pedestal/robot2_pedestal.xacro (robot description, xacro)
@@ -3,5 +3,5 @@
   xmlns:xacro="http://www.ros.org/wiki/xacro">
   <xacro:arg name="pedestal_prefix" default="robot2"/>
-  <xacro:arg name="pedestal_parent" default="world"/>
+  <xacro:arg name="pedestal_parent" default="world_interface"/>
   <xacro:arg name="pedestal_height" default="0.5"/>
   <link name="world_interface"/>
