Commit message: Fix

File: hrwros_week3/hrwros_support/urdf/hrwros.xacro (robot description, xacro)
@@ -13,35 +13,35 @@
   <xacro:include filename="$(find hrwros_support)/urdf/break_beam/break_beam.urdf.xacro"/>
   <!-- paramaters -->
-  <xacro:arg name="robot1" default="robot1"/>
-  <xacro:arg name="robot2" default="robot2"/>
-  <xacro:arg name="ur_type1" default="ur10"/>
-  <xacro:arg name="ur_type2" default="ur5"/>
-  <xacro:arg name="pedestal1_height" default="0.95"/>
-  <xacro:arg name="pedestal2_height" default="0.5"/>
-  <xacro:arg name="vacuum_gripper1" default="vacuum_gripper1_"/>
-  <xacro:arg name="vacuum_gripper2" default="vacuum_gripper2_"/>
+  <xacro:property name="robot1" value="robot1"/>
+  <xacro:property name="robot2" value="robot2"/>
+  <xacro:property name="ur_type1" value="ur10"/>
+  <xacro:property name="ur_type2" value="ur5"/>
+  <xacro:property name="pedestal1_height" value="0.95"/>
+  <xacro:property name="pedestal2_height" value="0.5"/>
+  <xacro:property name="vacuum_gripper1" value="vacuum_gripper1_"/>
+  <xacro:property name="vacuum_gripper2" value="vacuum_gripper2_"/>
   <!-- Workcell -->
   <xacro:workcell_urdf workcell_parent_name="world_interface"/>
   <!-- Robots -->
   <!-- Robot1 Pedestal -->
-  <xacro:robot_pedestal_urdf pedestal_prefix="$(arg robot1)_" pedestal_parent="world_interface" pedestal_height="$(arg pedestal1_height)">
+  <xacro:robot_pedestal_urdf pedestal_prefix="${robot1}_" pedestal_parent="world_interface" pedestal_height="${pedestal1_height}">
     <origin xyz="0.5 1.8 0.0" rpy="0 0 0"/>
   </xacro:robot_pedestal_urdf>
   <!-- Robot1 -->
-  <xacro:ur_description robot_name="$(arg robot1)" ur_type="$(arg ur_type1)">
-    <origin xyz="0.0 0.0 $(arg pedestal1_height)" rpy="0 0 0"/>
+  <xacro:ur_description robot_name="${robot1}" ur_type="${ur_type1}">
+    <origin xyz="0.0 0.0 ${pedestal1_height}" rpy="0 0 0"/>
   </xacro:ur_description>
   <!-- Vacuum Gripper1 -->
-  <xacro:vacuum_gripper_urdf prefix="$(arg vacuum_gripper1)" />
+  <xacro:vacuum_gripper_urdf prefix="${vacuum_gripper1}" />
   <!-- Robot2 Pedestal -->
-  <xacro:robot_pedestal_urdf pedestal_prefix="$(arg robot2)_" pedestal_parent="world_interface" pedestal_height="$(arg pedestal2_height)">
+  <xacro:robot_pedestal_urdf pedestal_prefix="${robot2}_" pedestal_parent="world_interface" pedestal_height="${pedestal2_height}">
     <origin xyz="-7.8 -1.5 0.0" rpy="0 0 0"/>
   </xacro:robot_pedestal_urdf>
   <!-- Robot2 -->
-  <xacro:ur_description robot_name="$(arg robot2)" ur_type="$(arg ur_type2)">
-    <origin xyz="0.0 0.0 $(arg pedestal2_height)" rpy="0 0 0"/>
+  <xacro:ur_description robot_name="${robot2}" ur_type="${ur_type2}">
+    <origin xyz="0.0 0.0 ${pedestal2_height}" rpy="0 0 0"/>
   </xacro:ur_description>
   <!-- Vacuum Gripper2 -->
-  <xacro:vacuum_gripper_urdf prefix="$(arg vacuum_gripper2)" />
+  <xacro:vacuum_gripper_urdf prefix="${vacuum_gripper2}" />
   <!-- Bins -->
   <!-- Bin1 -->
@@ -63,5 +63,5 @@
   </xacro:break_beam_urdf>
   <!-- Joints -->
- <joint name="world_interface_to_world" type="fixed">
+  <joint name="world_interface_to_world" type="fixed">
     <parent link="world" />
     <child link="world_interface" />
@@ -69,11 +69,11 @@
   <!-- gripper1 to robot1. -->
   <joint name="gripper1_to_robot1" type="fixed">
-    <parent link="$(arg robot1)_tool0" />
-    <child link="$(arg vacuum_gripper1)base_link" />
+    <parent link="${robot1}_tool0" />
+    <child link="${vacuum_gripper1}base_link" />
   </joint>
   <!-- gripper2 to robot2. -->
   <joint name="gripper2_to_robot2" type="fixed">
-    <parent link="$(arg robot2)_tool0" />
-    <child link="$(arg vacuum_gripper2)base_link" />
+    <parent link="${robot2}_tool0" />
+    <child link="${vacuum_gripper2}base_link" />
   </joint>
   <joint name="bin_1_joint" type="fixed">

Commit message: Fix

File: hrwros_week3/hrwros_support/urdf/hrwros.xacro (robot description, xacro)
@@ -51,9 +51,9 @@
   <!-- Logical Cameras -->
   <!-- Logical Camera 1 -->
-  <xacro:logical_camera_urdf prefix="logical_camera1_">
+  <xacro:logical_camera_urdf prefix="logical_camera1_" logical_camera_parent="world_interface">
     <origin xyz="1.2 1.8 2.0" rpy="0 1.5708 0"/>
   </xacro:logical_camera_urdf>
   <!-- Logical Camera 2 -->
-  <xacro:logical_camera_urdf prefix="logical_camera2_">
+  <xacro:logical_camera_urdf prefix="logical_camera2_" logical_camera_parent="world_interface">
     <origin xyz="-8.3 -1.23 1.8" rpy="0 1.5708 0"/>
   </xacro:logical_camera_urdf>

File: hrwros_week3/hrwros_support/urdf/logical_camera/logical_camera.urdf.xacro (robot description, xacro)
@@ -1,12 +1,13 @@
 <?xml version="1.0"?>
-<robot name="logical_camera_urdf" xmlns:xacro="http://www.ros.org/wiki/xacro">
-  <xacro:macro name="logical_camera_urdf" params="prefix *origin">
+<robot name="logical_camera_urdf"
+  xmlns:xacro="http://www.ros.org/wiki/xacro">
+  <xacro:macro name="logical_camera_urdf" params="prefix logical_camera_parent *origin">
     <xacro:property name="length" value="0.2"/>
     <xacro:property name="width" value="0.050"/>
     <xacro:property name="height" value="0.050"/>
     <joint name="${prefix}logical_camera_joint" type="fixed">
-	<xacro:insert_block name="origin" />
-	<parent link="world_interface"/>
-	<child link="${prefix}base_link"/>
+      <xacro:insert_block name="origin" />
+      <parent link="${logical_camera_parent}"/>
+      <child link="${prefix}base_link"/>
     </joint>
     <!-- link list -->
@@ -30,7 +31,5 @@
       <inertial>
         <origin xyz="0 0 0" rpy="0 0 0" />
-        <inertia ixx="0.1" ixy="0" ixz="0"
-                 iyy="0.1" iyz="0"
-                 izz="0.1" />
+        <inertia ixx="0.1" ixy="0" ixz="0" iyy="0.1" iyz="0" izz="0.1" />
         <mass value="1" />
       </inertial>

File: hrwros_week3/hrwros_support/urdf/logical_camera/logical_camera1.xacro (robot description, xacro)
@@ -3,7 +3,8 @@
   xmlns:xacro="http://www.ros.org/wiki/xacro">
   <xacro:arg name="prefix" default="logical_camera1_"/>
+  <link name="world_interface"/>
   <!-- URDF -->
   <xacro:include filename="$(find hrwros_support)/urdf/logical_camera/logical_camera.urdf.xacro"/>
-  <xacro:logical_camera_urdf prefix="$(arg prefix)">
+  <xacro:logical_camera_urdf prefix="$(arg prefix)" logical_camera_parent="$(arg logical_camera_parent)">
     <origin xyz="1.2 1.8 2.0" rpy="0 1.5708 0"/>
   </xacro:logical_camera_urdf>

File: hrwros_week3/hrwros_support/urdf/logical_camera/logical_camera2.xacro (robot description, xacro)
@@ -3,7 +3,9 @@
   xmlns:xacro="http://www.ros.org/wiki/xacro">
   <xacro:arg name="prefix" default="logical_camera2_"/>
+  <xacro:arg name="logical_camera_parent" default="world_interface"/>
+  <link name="world_interface"/>
   <!-- URDF -->
   <xacro:include filename="$(find hrwros_support)/urdf/logical_camera/logical_camera.urdf.xacro"/>
-  <xacro:logical_camera_urdf prefix="logical_camera2_">
+  <xacro:logical_camera_urdf prefix="$(arg prefix)" logical_camera_parent="$(arg logical_camera_parent)">
     <origin xyz="-8.3 -1.23 1.8" rpy="0 1.5708 0"/>
   </xacro:logical_camera_urdf>
