Commit message: fix hrwros_support/

File: hrwros_week3/hrwros_support/urdf/bin/bin.urdf.xacro (robot description, xacro)
@@ -3,5 +3,5 @@
   <xacro:macro name="bin_urdf" params="prefix parent *origin">
     <!-- link list -->
-    <link name="${prefix}_base_link">
+    <link name="${prefix}base_link">
       <visual>
         <origin xyz="0 0 0" rpy="0 0 0" />
@@ -28,5 +28,5 @@
       </inertial>
     </link>
-    <link name="${prefix}_drop_point">
+    <link name="${prefix}drop_point">
       <inertial>
         <origin xyz="0 0 0" rpy="0 0 0" />
@@ -36,13 +36,13 @@
     </link>
     <!-- joint list -->
-    <joint name="${prefix}_joint_1" type="fixed">
+    <joint name="${prefix}joint_1" type="fixed">
       <parent link="${parent}" />
-      <child link="${prefix}_base_link" />
+      <child link="${prefix}base_link" />
       <xacro:insert_block name="origin" />
     </joint>
-    <joint name="${prefix}_joint_2" type="fixed">
+    <joint name="${prefix}joint_2" type="fixed">
       <origin xyz="0 0 1.0" rpy="0 0 0" />
-      <parent link="${prefix}_base_link" />
-      <child link="${prefix}_drop_point" />
+      <parent link="${prefix}base_link" />
+      <child link="${prefix}drop_point" />
     </joint>
   </xacro:macro>

File: hrwros_week3/hrwros_support/urdf/hrwros.xacro (robot description, xacro)
@@ -22,5 +22,5 @@
   <!-- Bins -->
   <!-- Bin1 -->
-  <xacro:bin_urdf prefix="bin_1" parent="world">
+  <xacro:bin_urdf prefix="bin_1_" parent="world">
     <origin xyz="-7.6 -1.7 0" rpy="0 0 0" />
   </xacro:bin_urdf>

Commit message: fix urdf support

File: hrwros_week3/hrwros_support/urdf/bin/bin.urdf.xacro (robot description, xacro)
@@ -1,5 +1,5 @@
 <?xml version="1.0"?>
 <robot xmlns:xacro="http://www.ros.org/wiki/xacro">
-  <xacro:macro name="bin_urdf" params="prefix parent *origin">
+  <xacro:macro name="bin_urdf" params="prefix *origin">
     <!-- link list -->
     <link name="${prefix}base_link">
@@ -37,5 +37,5 @@
     <!-- joint list -->
     <joint name="${prefix}joint_1" type="fixed">
-      <parent link="${parent}" />
+      <parent link="world" />
       <child link="${prefix}base_link" />
       <xacro:insert_block name="origin" />

File: hrwros_week3/hrwros_support/urdf/break_beam/break_beam.urdf.xacro (robot description, xacro)
@@ -2,7 +2,7 @@
 <robot name="break_beam_urdf"
   xmlns:xacro="http://www.ros.org/wiki/xacro">
-  <xacro:macro name="break_beam_urdf" params="prefix parent *origin">
+  <xacro:macro name="break_beam_urdf" params="prefix *origin">
     <!-- link list -->
-    <link name="${prefix}${parent}"/>
+    <link name="${prefix}world"/>
     <link name="${prefix}base_link">
       <visual>
@@ -29,12 +29,11 @@
     </link>
     <link name="${prefix}optical_link"/>
-    <!-- external parent joint -->
-    <joint name="${prefix}break_beam_joint" type="fixed">
-      <parent link="${parent}" />
-      <child link="${prefix}${parent}" />
+    <!-- joint list -->
+    <joint name="${prefix}joint" type="fixed">
+      <parent link="world" />
+      <child link="${prefix}world" />
     </joint>
-    <!-- joint list -->
     <joint name="${prefix}world_joint" type="fixed">
-      <parent link="${prefix}${parent}" />
+      <parent link="${prefix}world" />
       <child link="${prefix}base_link" />
       <xacro:insert_block name="origin" />

File: hrwros_week3/hrwros_support/urdf/break_beam/break_beam.xacro (robot description, xacro)
@@ -2,10 +2,9 @@
 <robot name="break_beam" xmlns:xacro="http://www.ros.org/wiki/xacro">
   <xacro:arg name="prefix" default="break_beam_"/>
-  <xacro:arg name="parent" default="world"/>
   <!-- URDF -->
   <xacro:include filename="$(find hrwros_support)/urdf/break_beam/break_beam.urdf.xacro"/>
-  <xacro:break_beam_urdf prefix="$(arg prefix)" parent="$(arg parent)"/>
+  <xacro:break_beam_urdf prefix="$(arg prefix)"/>
   <!-- Gazebo -->
   <xacro:include filename="$(find hrwros_support)/urdf/break_beam/break_beam.gazebo.xacro"/>
-  <xacro:break_beam_gazebo prefix="$(arg prefix)" parent="$(arg parent)"/>
+  <xacro:break_beam_gazebo prefix="$(arg prefix)"/>
 </robot>

File: hrwros_week3/hrwros_support/urdf/hrwros.xacro (robot description, xacro)
@@ -1,40 +1,75 @@
 <?xml version="1.0" ?>
-<robot name="robot" xmlns:xacro="http://www.ros.org/wiki/xacro">
+<robot name="robot"
+  xmlns:xacro="http://www.ros.org/wiki/xacro">
   <!-- world -->
   <link name="world" />
   <!-- Include necessary URDF files from hrwros_support -->
+  <xacro:include filename="$(find hrwros_support)/urdf/robot_pedestal/robot_pedestal.urdf.xacro"/>
+  <xacro:include filename="$(find hrwros_support)/urdf/arm_robot/ur_description.urdf.xacro"/>
+  <xacro:include filename="$(find hrwros_support)/urdf/vacuum_gripper/vacuum_gripper.urdf.xacro"/>
   <xacro:include filename="$(find hrwros_support)/urdf/workcell/workcell.urdf.xacro"/>
-  <xacro:include filename="$(find hrwros_support)/urdf/container_arm_robot_pedestal/container_arm_robot_pedestal.urdf.xacro"/>
   <xacro:include filename="$(find hrwros_support)/urdf/bin/bin.urdf.xacro"/>
   <xacro:include filename="$(find hrwros_support)/urdf/logical_camera/logical_camera.urdf.xacro"/>
   <xacro:include filename="$(find hrwros_support)/urdf/break_beam/break_beam.urdf.xacro"/>
+  <!-- paramaters -->
+  <xacro:arg name="robot1" default="robot1"/>
+  <xacro:arg name="robot2" default="robot2"/>
+  <xacro:arg name="ur_type1" default="ur10"/>
+  <xacro:arg name="ur_type2" default="ur5"/>
+  <xacro:arg name="pedestal1_height" default="0.95"/>
+  <xacro:arg name="pedestal2_height" default="0.5"/>
+  <xacro:arg name="vacuum_gripper1" default="vacuum_gripper1_"/>
+  <xacro:arg name="vacuum_gripper2" default="vacuum_gripper2_"/>
   <!-- Workcell -->
-  <xacro:workcell_urdf parent="world"/>
+  <xacro:workcell_urdf workcell_parent_name="world"/>
   <!-- Robots -->
+  <!-- Robot1 Pedestal -->
+  <xacro:robot_pedestal_urdf pedestal_prefix="$(arg robot1)_" pedestal_parent="world" pedestal_height="$(arg pedestal1_height)">
+    <origin xyz="0.5 1.8 0.0" rpy="0 0 0"/>
+  </xacro:robot_pedestal_urdf>
   <!-- Robot1 -->
-  <xacro:container_arm_robot_pedestal_urdf robot_name="robot1" ur_type="ur10" parent_pedestal="world" height_pedestal="0.95">
-    <origin xyz="0.5 1.8 0.0" rpy="0 0 0"/>
-  </xacro:container_arm_robot_pedestal_urdf>
+  <xacro:ur_description robot_name="$(arg robot1)" ur_type="$(arg ur_type1)">
+    <origin xyz="0.0 0.0 $(arg pedestal1_height)" rpy="0 0 0"/>
+  </xacro:ur_description>
+  <!-- Vacuum Gripper1 -->
+  <xacro:vacuum_gripper_urdf prefix="$(arg vacuum_gripper1)" joint_prefix="$(arg vacuum_gripper1)joint"/>
+  <!-- Robot2 Pedestal -->
+  <xacro:robot_pedestal_urdf pedestal_prefix="$(arg robot2)_" pedestal_parent="world" pedestal_height="$(arg pedestal2_height)">
+    <origin xyz="-7.6 -0.5 0.0" rpy="0 0 0"/>
+  </xacro:robot_pedestal_urdf>
   <!-- Robot2 -->
-  <xacro:container_arm_robot_pedestal_urdf robot_name="robot2" ur_type="ur10" parent_pedestal="world" height_pedestal="0.5">
-    <origin xyz="-7.6 -0.5 0.0" rpy="0 0 0"/>
-  </xacro:container_arm_robot_pedestal_urdf>
+  <xacro:ur_description robot_name="$(arg robot2)" ur_type="$(arg ur_type2)">
+    <origin xyz="0.0 0.0 $(arg pedestal2_height)" rpy="0 0 0"/>
+  </xacro:ur_description>
+  <!-- Vacuum Gripper2 -->
+  <xacro:vacuum_gripper_urdf prefix="$(arg vacuum_gripper2)" joint_prefix="$(arg vacuum_gripper2)joint"/>
   <!-- Bins -->
   <!-- Bin1 -->
-  <xacro:bin_urdf prefix="bin_1_" parent="world">
+  <xacro:bin_urdf prefix="bin_1_">
     <origin xyz="-7.6 -1.7 0" rpy="0 0 0" />
   </xacro:bin_urdf>
   <!-- Logical Cameras -->
   <!-- Logical Camera 1 -->
-  <xacro:logical_camera_urdf prefix="logical_camera1_" logical_camera_parent="world">
+  <xacro:logical_camera_urdf prefix="logical_camera1_">
     <origin xyz="1.2 1.8 2.0" rpy="0 1.5708 0"/>
   </xacro:logical_camera_urdf>
   <!-- Logical Camera 2 -->
-  <xacro:logical_camera_urdf prefix="logical_camera2_" logical_camera_parent="world">
+  <xacro:logical_camera_urdf prefix="logical_camera2_">
     <origin xyz="-8.3 -1.23 1.8" rpy="0 1.5708 0"/>
   </xacro:logical_camera_urdf>
   <!-- Break Beam -->
-  <xacro:break_beam_urdf prefix="break_beam_" parent="world">
+  <xacro:break_beam_urdf prefix="break_beam_">
     <origin xyz="1.6 1.9 0.925" rpy="0 0 ${radians(180)}" />
   </xacro:break_beam_urdf>
+  <!-- Joints -->
+  <!-- gripper1 to robot1. -->
+  <joint name="gripper1_to_robot1" type="fixed">
+    <parent link="$(arg robot1)_tool0" />
+    <child link="$(arg vacuum_gripper1)base_link" />
+  </joint>
+  <!-- gripper2 to robot2. -->
+  <joint name="gripper2_to_robot2" type="fixed">
+    <parent link="$(arg robot2)_tool0" />
+    <child link="$(arg vacuum_gripper2)base_link" />
+  </joint>
 </robot>

File: hrwros_week3/hrwros_support/urdf/logical_camera/logical_camera.urdf.xacro (robot description, xacro)
@@ -1,5 +1,5 @@
 <?xml version="1.0"?>
 <robot name="logical_camera_urdf" xmlns:xacro="http://www.ros.org/wiki/xacro">
-  <xacro:macro name="logical_camera_urdf" params="prefix logical_camera_parent *origin">
+  <xacro:macro name="logical_camera_urdf" params="prefix *origin">
     <xacro:property name="length" value="0.2"/>
     <xacro:property name="width" value="0.050"/>
@@ -7,5 +7,5 @@
     <joint name="${prefix}logical_camera_joint" type="fixed">
 	<xacro:insert_block name="origin" />
-	<parent link="${logical_camera_parent}"/>
+	<parent link="world"/>
 	<child link="${prefix}base_link"/>
     </joint>

File: hrwros_week3/hrwros_support/urdf/robot_pedestal/robot_pedestal.urdf.xacro (robot description, xacro)
@@ -2,6 +2,6 @@
 <robot name="robot_pedestal_urdf" xmlns:xacro="http://www.ros.org/wiki/xacro">
 <!-- robot pedestal -->
-<xacro:macro name = "robot_pedestal_urdf" params = "prefix parent pedestal_height *origin">
-  <link name="${prefix}_pedestal_link">
+<xacro:macro name = "robot_pedestal_urdf" params = "pedestal_prefix pedestal_parent pedestal_height *origin">
+  <link name="${pedestal_prefix}pedestal_link">
     <visual>
       <origin xyz="0 0 ${0.5*pedestal_height}"/>
@@ -25,10 +25,10 @@
     </inertial>
   </link>
-  <joint name="${prefix}_pedestal_joint" type="fixed">
+  <joint name="${pedestal_prefix}pedestal_joint" type="fixed">
     <xacro:insert_block name="origin" />
-    <parent link="${parent}"/>
-    <child link="${prefix}_pedestal_link"/>
+    <parent link="${pedestal_parent}"/>
+    <child link="${pedestal_prefix}pedestal_link"/>
   </joint>
-  <gazebo reference="${prefix}_pedestal_link">
+  <gazebo reference="${pedestal_prefix}pedestal_link">
     <material>Gazebo/Blue</material>
   </gazebo>

File: hrwros_week3/hrwros_support/urdf/vacuum_gripper/vacuum_gripper.urdf.xacro (robot description, xacro)
@@ -1,7 +1,7 @@
 <?xml version="1.0"?>
 <robot xmlns:xacro="http://www.ros.org/wiki/xacro">
-  <xacro:macro name="vacuum_gripper_urdf" params="prefix parent">
+  <xacro:macro name="vacuum_gripper_urdf" params="prefix joint_prefix">
     <!-- link list -->
-    <link name="${prefix}_vacuum_gripper_base_link" >
+    <link name="${prefix}base_link">
       <visual>
         <origin xyz="0 0 0" rpy="0 0 0" />
@@ -22,11 +22,9 @@
       <inertial>
         <origin xyz="0 0 0" rpy="0 0 0" />
-        <inertia ixx="1.0" ixy="0" ixz="0"
-                 iyy="1.0" iyz="0"
-                 izz="1.0" />
+        <inertia ixx="1.0" ixy="0" ixz="0" iyy="1.0" iyz="0" izz="1.0" />
         <mass value="1.0" />
       </inertial>
     </link>
-    <link name="${prefix}_vacuum_gripper_suction_cup">
+    <link name="${prefix}suction_cup">
       <visual>
         <origin xyz="0 0 0" rpy="0 0 0" />
@@ -47,19 +45,13 @@
       <inertial>
         <origin xyz="0 0 0" rpy="0 0 0" />
-        <inertia ixx="0.0001" ixy="0" ixz="0"
-                 iyy="0.0001" iyz="0"
-                 izz="0.0001" />
+        <inertia ixx="0.0001" ixy="0" ixz="0" iyy="0.0001" iyz="0" izz="0.0001" />
         <mass value="0.00001" />
       </inertial>
     </link>
     <!-- joint list -->
-  <joint name="${prefix}_to_vacuum_gripper_joint_1" type="fixed">
-    <parent link="${parent}" />
-    <child link="${prefix}_vacuum_gripper_base_link" />
-  </joint>
-    <joint name="${prefix}_to_vacuum_gripper_joint_2" type="fixed">
+    <joint name="${joint_prefix}" type="fixed">
       <origin xyz="0 0 0.01" rpy="0 0 0" />
-      <parent link="${prefix}_vacuum_gripper_base_link"  />
-      <child link="${prefix}_vacuum_gripper_suction_cup" />
+      <parent link="${prefix}base_link" />
+      <child link="${prefix}suction_cup" />
     </joint>
   </xacro:macro>

File: hrwros_week3/hrwros_support/urdf/workcell/workcell.urdf.xacro (robot description, xacro)
@@ -1,5 +1,5 @@
 <?xml version="1.0" ?>
 <robot name="workcell_urdf" xmlns:xacro="http://www.ros.org/wiki/xacro">
-    <xacro:macro name="workcell_urdf" params="parent">
+    <xacro:macro name="workcell_urdf" params="workcell_parent_name">
     <!-- Links -->
     <link name="workcell">
@@ -21,6 +21,6 @@
       </inertial>
     </link>
-    <joint name="workcell_to_${parent}" type="fixed">
-      <parent link="${parent}" />
+    <joint name="workcell_to_${workcell_parent_name}" type="fixed">
+      <parent link="${workcell_parent_name}" />
       <child link="workcell" />
       <origin xyz="0 0 0" rpy="0 0 ${radians(90)}" />

Commit message: fix

File: hrwros_week3/hrwros_support/urdf/bin/bin.urdf.xacro (robot description, xacro)
@@ -36,9 +36,4 @@
     </link>
     <!-- joint list -->
-    <joint name="${prefix}joint_1" type="fixed">
-      <parent link="world" />
-      <child link="${prefix}base_link" />
-      <xacro:insert_block name="origin" />
-    </joint>
     <joint name="${prefix}joint_2" type="fixed">
       <origin xyz="0 0 1.0" rpy="0 0 0" />

File: hrwros_week3/hrwros_support/urdf/hrwros.xacro (robot description, xacro)
@@ -77,4 +77,9 @@
     <child link="$(arg vacuum_gripper2)base_link" />
   </joint>
+  <joint name="bin_1_joint" type="fixed">
+    <parent link="world_interface" />
+    <child link="bin_1_base_link" />
+    <origin xyz="-8.0 -2.2 0.0" rpy="0 0 0" />
+  </joint>
   <!-- break beam to world. -->
   <joint name="break_beam_joint" type="fixed">

File: hrwros_week3/hrwros_support/urdf/robot_pedestal/robot1_pedestal.xacro (robot description, xacro)
@@ -4,4 +4,5 @@
   <xacro:arg name="pedestal_parent" default="world"/>
   <xacro:arg name="pedestal_height" default="0.95"/>
+  <link name="world_interface"/>
   <!-- URDF -->
   <xacro:include filename="$(find hrwros_support)/urdf/robot_pedestal/robot_pedestal.urdf.xacro"/>

File: hrwros_week3/hrwros_support/urdf/robot_pedestal/robot2_pedestal.xacro (robot description, xacro)
@@ -1,7 +1,9 @@
 <?xml version="1.0" ?>
-<robot name="robot2_pedestal" xmlns:xacro="http://www.ros.org/wiki/xacro">
+<robot name="robot2_pedestal"
+  xmlns:xacro="http://www.ros.org/wiki/xacro">
   <xacro:arg name="pedestal_prefix" default="robot2"/>
   <xacro:arg name="pedestal_parent" default="world"/>
   <xacro:arg name="pedestal_height" default="0.5"/>
+  <link name="world_interface"/>
   <!-- URDF -->
   <xacro:include filename="$(find hrwros_support)/urdf/robot_pedestal/robot_pedestal.urdf.xacro"/>

Commit message: Fix spawn mesh

File: hrwros_week3/hrwros_support/urdf/bin/bin.urdf.xacro (robot description, xacro)
@@ -7,5 +7,5 @@
         <origin xyz="0 0 0" rpy="0 0 0" />
         <geometry>
-          <mesh filename="package://hrwros_support/meshes/bin/visual/bin.dae" />
+          <mesh filename="file://$(find hrwros_support)/meshes/bin/visual/bin.dae"/>
         </geometry>
       </visual>
@@ -13,5 +13,5 @@
         <origin xyz="0 0 0" rpy="0 0 0"/>
         <geometry>
-          <mesh filename="package://hrwros_support/meshes/bin/collision/bin_bottom.dae"/>
+          <mesh filename="file://$(find hrwros_support)/meshes/bin/collision/bin_bottom.dae"/>
         </geometry>
       </collision>
@@ -19,5 +19,5 @@
         <origin xyz="0 0 0" rpy="0 0 0"/>
         <geometry>
-          <mesh filename="package://hrwros_support/meshes/bin/collision/bin_sides.dae"/>
+          <mesh filename="file://$(find hrwros_support)/meshes/bin/collision/bin_sides.dae"/>
         </geometry>
       </collision>

File: hrwros_week3/hrwros_support/urdf/break_beam/break_beam.urdf.xacro (robot description, xacro)
@@ -9,5 +9,5 @@
         <origin xyz="0 0 0" rpy="0 0 0" />
         <geometry>
-          <mesh filename="package://hrwros_support/meshes/break_beam/visual/hokuyo.dae" />
+          <mesh filename="file://$(find hrwros_support)/meshes/break_beam/visual/hokuyo.dae"/>
         </geometry>
         <material name="dark_grey">
@@ -18,5 +18,5 @@
         <origin xyz="0 0 0" rpy="0 0 0" />
         <geometry>
-          <mesh filename="package://hrwros_support/meshes/break_beam/collision/hokuyo.dae" />
+          <mesh filename="file://$(find hrwros_support)/meshes/break_beam/collision/hokuyo.dae"/>
         </geometry>
         <material name="dark_grey"/>

File: hrwros_week3/hrwros_support/urdf/vacuum_gripper/vacuum_gripper.urdf.xacro (robot description, xacro)
@@ -8,5 +8,5 @@
         <origin xyz="0 0 0" rpy="0 0 0" />
         <geometry>
-          <mesh filename="package://hrwros_support/meshes/vacuum_gripper/visual/vacuum_gripper.dae"/>
+          <mesh filename="file://$(find hrwros_support)/meshes/vacuum_gripper/visual/vacuum_gripper.dae"/>
         </geometry>
         <material name="red">
@@ -17,5 +17,5 @@
         <origin xyz="0 0 0" rpy="0 0 0"/>
         <geometry>
-          <mesh filename="package://hrwros_support/meshes/vacuum_gripper/collision/vacuum_gripper.dae"/>
+          <mesh filename="file://$(find hrwros_support)/meshes/vacuum_gripper/collision/vacuum_gripper.dae"/>
         </geometry>
         <material name="red"/>

File: hrwros_week3/hrwros_support/urdf/workcell/workcell.urdf.xacro (robot description, xacro)
@@ -7,10 +7,10 @@
       <visual>
         <geometry>
-          <mesh filename="package://hrwros_support/meshes/workcell/visual/workcell.dae"/>
+          <mesh filename="file://$(find hrwros_support)/meshes/workcell/visual/workcell.dae"/>
         </geometry>
       </visual>
       <collision>
         <geometry>
-          <mesh filename="package://hrwros_support/meshes/workcell/collision/workcell.dae"/>
+          <mesh filename="file://$(find hrwros_support)/meshes/workcell/collision/workcell.dae"/>
         </geometry>
       </collision>
