Commit message: fix urdf support

File: hrwros_week3/hrwros_support/urdf/bin/bin.xacro (robot description, xacro)
@@ -1,8 +1,11 @@
 <?xml version="1.0"?>
-<robot name="bin" xmlns:xacro="http://www.ros.org/wiki/xacro">
+<robot name="bin"
+  xmlns:xacro="http://www.ros.org/wiki/xacro">
   <xacro:arg name="prefix" default="bin_1_"/>
   <!-- URDF -->
   <xacro:include filename="$(find hrwros_support)/urdf/bin/bin.urdf.xacro"/>
-  <xacro:bin_urdf prefix="$(arg prefix)"/>
+  <xacro:bin_urdf prefix="$(arg prefix)">
+    <origin xyz="-8.0 -2.2 0.0" rpy="0 0 0" />
+  </xacro:bin_urdf>
   <!-- Gazebo -->
   <xacro:include filename="$(find hrwros_support)/urdf/bin/bin.gazebo.xacro"/>

File: hrwros_week3/hrwros_support/urdf/break_beam/break_beam.xacro (robot description, xacro)
@@ -1,8 +1,11 @@
 <?xml version="1.0"?>
-<robot name="break_beam" xmlns:xacro="http://www.ros.org/wiki/xacro">
+<robot name="break_beam"
+  xmlns:xacro="http://www.ros.org/wiki/xacro">
   <xacro:arg name="prefix" default="break_beam_"/>
   <!-- URDF -->
   <xacro:include filename="$(find hrwros_support)/urdf/break_beam/break_beam.urdf.xacro"/>
-  <xacro:break_beam_urdf prefix="$(arg prefix)"/>
+  <xacro:break_beam_urdf prefix="$(arg prefix)">
+    <origin xyz="1.6 1.9 0.925" rpy="0 0 ${radians(180)}" />
+  </xacro:break_beam_urdf>
   <!-- Gazebo -->
   <xacro:include filename="$(find hrwros_support)/urdf/break_beam/break_beam.gazebo.xacro"/>

File: hrwros_week3/hrwros_support/urdf/hrwros.xacro (robot description, xacro)
@@ -33,8 +33,8 @@
   </xacro:ur_description>
   <!-- Vacuum Gripper1 -->
-  <xacro:vacuum_gripper_urdf prefix="$(arg vacuum_gripper1)" joint_prefix="$(arg vacuum_gripper1)joint"/>
+  <xacro:vacuum_gripper_urdf prefix="$(arg vacuum_gripper1)" />
   <!-- Robot2 Pedestal -->
   <xacro:robot_pedestal_urdf pedestal_prefix="$(arg robot2)_" pedestal_parent="world" pedestal_height="$(arg pedestal2_height)">
-    <origin xyz="-7.6 -0.5 0.0" rpy="0 0 0"/>
+    <origin xyz="-7.8 -1.5 0.0" rpy="0 0 0"/>
   </xacro:robot_pedestal_urdf>
   <!-- Robot2 -->
@@ -43,9 +43,9 @@
   </xacro:ur_description>
   <!-- Vacuum Gripper2 -->
-  <xacro:vacuum_gripper_urdf prefix="$(arg vacuum_gripper2)" joint_prefix="$(arg vacuum_gripper2)joint"/>
+  <xacro:vacuum_gripper_urdf prefix="$(arg vacuum_gripper2)" />
   <!-- Bins -->
   <!-- Bin1 -->
   <xacro:bin_urdf prefix="bin_1_">
-    <origin xyz="-7.6 -1.7 0" rpy="0 0 0" />
+    <origin xyz="-8.0 -2.2 0.0" rpy="0 0 0" />
   </xacro:bin_urdf>
   <!-- Logical Cameras -->

File: hrwros_week3/hrwros_support/urdf/vacuum_gripper/vacuum_gripper.urdf.xacro (robot description, xacro)
@@ -1,5 +1,6 @@
 <?xml version="1.0"?>
 <robot xmlns:xacro="http://www.ros.org/wiki/xacro">
-  <xacro:macro name="vacuum_gripper_urdf" params="prefix joint_prefix">
+  <xacro:macro name="vacuum_gripper_urdf" params="prefix">
+    <xacro:property name="joint_prefix" value="${prefix}joint"/>
     <!-- link list -->
     <link name="${prefix}base_link">

Commit message: update spawn_turtlebot

File: hrwros_week3/hrwros_support/urdf/bin/bin.xacro (robot description, xacro)
@@ -8,5 +8,6 @@
   <xacro:include filename="$(find hrwros_support)/urdf/bin/bin.urdf.xacro"/>
   <xacro:bin_urdf prefix="$(arg prefix)" bin_parent="$(arg bin_parent)">
-    <origin xyz="-8.0 -2.2 0.0" rpy="0 0 0" />
+    <!-- <origin xyz="-8.0 -2.2 0.0" rpy="0 0 0" /> -->
+    <origin xyz="0.0 0.0 0.0" rpy="0 0 0" />
   </xacro:bin_urdf>
   <!-- Gazebo -->
