Commit message: Working on spawn_robots.launch.py

File: hrwros_week3/hrwros_support/urdf/robot_system/robot_system.urdf.xacro (robot description, xacro)
@@ -11,4 +11,5 @@
     <xacro:ur_description robot_name="${robot_prefix}" ur_type="${robot_type}">
       <!-- <origin xyz="0.0 0.0 ${pedestal1_height}" rpy="0 0 0"/> -->
+      <origin xyz="0.0 0.0 0.0" rpy="0 0 0"/>
     </xacro:ur_description>
     <!-- Vacuum Gripper1 -->

Commit message: Working on spawn_robots.launch.py

File: hrwros_week3/hrwros_support/urdf/robot_system/robot_system.urdf.xacro (robot description, xacro)
@@ -7,5 +7,5 @@
     <xacro:include filename="$(find hrwros_support)/urdf/vacuum_gripper/vacuum_gripper.urdf.xacro"/>
     <!-- Used for fixing robot to Gazebo 'base_link' -->
-    <link name="world"/>
+    <link name="world_interface"/>
     <!-- Robot1 -->
     <xacro:ur_description robot_name="${robot_prefix}" ur_type="${robot_type}">
