Commit message: Working on spawn_robots.launch.py

File: hrwros_week3/hrwros_support/urdf/arm_robot/ur_description.urdf.xacro (robot description, xacro)
@@ -18,5 +18,5 @@
         name="${robot_name}"
         tf_prefix="${tf_prefix}"
-        parent="${robot_name}_pedestal_link"
+        parent="world_interface"
         joint_limits_parameters_file="${joint_limit_params}"
         kinematics_parameters_file="${kinematics_params}"

File: hrwros_week3/hrwros_support/urdf/hrwros.xacro (robot description, xacro)
@@ -30,5 +30,5 @@
   <!-- Robot1 -->
   <xacro:ur_description robot_name="${robot1}" ur_type="${ur_type1}">
-    <origin xyz="0.0 0.0 ${pedestal1_height}" rpy="0 0 0"/>
+    <origin xyz="0.5 1.8 ${pedestal1_height}" rpy="0 0 0"/>
   </xacro:ur_description>
   <!-- Vacuum Gripper1 -->
@@ -40,5 +40,5 @@
   <!-- Robot2 -->
   <xacro:ur_description robot_name="${robot2}" ur_type="${ur_type2}">
-    <origin xyz="0.0 0.0 ${pedestal2_height}" rpy="0 0 0"/>
+    <origin xyz="-7.8 -1.5 ${pedestal2_height}" rpy="0 0 0"/>
   </xacro:ur_description>
   <!-- Vacuum Gripper2 -->

Commit message: Add my_python_utils

File: hrwros_week3/hrwros_support/urdf/arm_robot/ur_description.urdf.xacro (robot description, xacro)
@@ -1,79 +1,44 @@
 <?xml version="1.0"?>
 <robot xmlns:xacro="http://www.ros.org/wiki/xacro">
-    <xacro:include filename="$(find ur_description)/urdf/ur_macro.xacro"/>
-    <xacro:include filename="$(find hrwros_support)/urdf/arm_robot/ur_params.urdf.xacro"/>
-    <!-- Custom Arm Robot Macro Definition -->
-    <xacro:macro name="ur_description" params="robot_name ur_type *origin">
-      <!-- parameters -->
-      <xacro:ur_params/>
-      <xacro:property name="tf_prefix" value="${robot_name}_"/>
-      <xacro:property name="joint_limit_params" default="$(find ur_description)/config/${ur_type}/joint_limits.yaml"/>
-      <xacro:property name="kinematics_params" default="$(find ur_description)/config/${ur_type}/default_kinematics.yaml"/>
-      <xacro:property name="physical_params" default="$(find ur_description)/config/${ur_type}/physical_parameters.yaml"/>
-      <xacro:property name="visual_params" default="$(find ur_description)/config/${ur_type}/visual_parameters.yaml"/>
-      <!-- convert to property to use substitution in function -->
-      <xacro:property name="initial_positions_file" value="$(arg initial_positions_file)"/>
-      <!-- Main robot arm setup -->
-      <xacro:ur_robot
-        name="${robot_name}"
-        tf_prefix="${tf_prefix}"
-        parent="world_interface"
-        joint_limits_parameters_file="${joint_limit_params}"
-        kinematics_parameters_file="${kinematics_params}"
-        physical_parameters_file="${physical_params}"
-        visual_parameters_file="${visual_params}"
-        transmission_hw_interface="$(arg transmission_hw_interface)"
-        safety_limits="$(arg safety_limits)"
-        safety_pos_margin="$(arg safety_pos_margin)"
-        safety_k_position="$(arg safety_k_position)"
-        use_fake_hardware="$(arg use_fake_hardware)"
-        fake_sensor_commands="$(arg fake_sensor_commands)"
-        sim_gazebo="$(arg sim_gazebo)"
-        sim_ignition="$(arg sim_ignition)"
-        headless_mode="$(arg headless_mode)"
-        initial_positions="${xacro.load_yaml(initial_positions_file)}"
-        use_tool_communication="$(arg use_tool_communication)"
-        tool_voltage="$(arg tool_voltage)"
-        tool_parity="$(arg tool_parity)"
-        tool_baud_rate="$(arg tool_baud_rate)"
-        tool_stop_bits="$(arg tool_stop_bits)"
-        tool_rx_idle_chars="$(arg tool_rx_idle_chars)"
-        tool_tx_idle_chars="$(arg tool_tx_idle_chars)"
-        tool_device_name="$(arg tool_device_name)"
-        tool_tcp_port="$(arg tool_tcp_port)"
-        robot_ip="$(arg robot_ip)"
-        script_filename="$(arg script_filename)"
-        output_recipe_filename="$(arg output_recipe_filename)"
-        input_recipe_filename="$(arg input_recipe_filename)"
-        reverse_ip="$(arg reverse_ip)"
-        script_command_port="$(arg script_command_port)"
-        reverse_port="$(arg reverse_port)"
-        script_sender_port="$(arg script_sender_port)"
-        trajectory_port="$(arg trajectory_port)"
-        >
-         <xacro:insert_block name="origin" />
-      </xacro:ur_robot>
-      <!-- Conditional inclusion for Gazebo simulation setup -->
-      <xacro:if value="$(arg sim_gazebo)">
-        <!-- Gazebo plugins -->
-        <gazebo reference="world">
-        </gazebo>
-        <gazebo>
-          <plugin filename="libgazebo_ros2_control.so" name="gazebo_ros2_control">
-            <parameters>$(arg simulation_controllers)</parameters>
-          </plugin>
-        </gazebo>
-      </xacro:if>
-      <xacro:if value="$(arg sim_ignition)">
-        <!-- Gazebo plugins -->
-        <gazebo reference="world">
-        </gazebo>
-        <gazebo>
-          <plugin filename="libign_ros2_control-system.so" name="ign_ros2_control::IgnitionROS2ControlPlugin">
-            <parameters>$(arg simulation_controllers)</parameters>
-            <controller_manager_node_name>$(arg tf_prefix)controller_manager</controller_manager_node_name>
-          </plugin>
-        </gazebo>
-      </xacro:if>
-    </xacro:macro>
+  <!-- /opt/ros/humble/share/ur_description/urdf/ -->
+  <xacro:include filename="$(find ur_description)/urdf/ur_macro.xacro"/>
+  <xacro:include filename="$(find hrwros_support)/urdf/arm_robot/ur_params.urdf.xacro"/>
+  <!-- Custom Arm Robot Macro Definition -->
+  <xacro:macro name="ur_description" params="robot_name robot_parent ur_type *origin">
+    <!-- parameters -->
+    <xacro:ur_params/>
+    <xacro:property name="tf_prefix" value="${robot_name}_"/>
+    <xacro:property name="joint_limit_params" default="$(find ur_description)/config/${ur_type}/joint_limits.yaml"/>
+    <xacro:property name="kinematics_params" default="$(find ur_description)/config/${ur_type}/default_kinematics.yaml"/>
+    <xacro:property name="physical_params" default="$(find ur_description)/config/${ur_type}/physical_parameters.yaml"/>
+    <xacro:property name="visual_params" default="$(find ur_description)/config/${ur_type}/visual_parameters.yaml"/>
+    <!-- convert to property to use substitution in function -->
+    <xacro:property name="initial_positions_file" value="$(arg initial_positions_file)"/>
+    <!-- Main robot arm setup -->
+    <xacro:ur_robot name="${robot_name}" tf_prefix="${tf_prefix}" parent="${robot_parent}" joint_limits_parameters_file="${joint_limit_params}" kinematics_parameters_file="${kinematics_params}" physical_parameters_file="${physical_params}" visual_parameters_file="${visual_params}" transmission_hw_interface="$(arg transmission_hw_interface)" safety_limits="$(arg safety_limits)" safety_pos_margin="$(arg safety_pos_margin)" safety_k_position="$(arg safety_k_position)" use_fake_hardware="$(arg use_fake_hardware)" fake_sensor_commands="$(arg fake_sensor_commands)" sim_gazebo="$(arg sim_gazebo)" sim_ignition="$(arg sim_ignition)" headless_mode="$(arg headless_mode)" initial_positions="${xacro.load_yaml(initial_positions_file)}" use_tool_communication="$(arg use_tool_communication)" tool_voltage="$(arg tool_voltage)" tool_parity="$(arg tool_parity)" tool_baud_rate="$(arg tool_baud_rate)" tool_stop_bits="$(arg tool_stop_bits)" tool_rx_idle_chars="$(arg tool_rx_idle_chars)" tool_tx_idle_chars="$(arg tool_tx_idle_chars)" tool_device_name="$(arg tool_device_name)" tool_tcp_port="$(arg tool_tcp_port)" robot_ip="$(arg robot_ip)" script_filename="$(arg script_filename)" output_recipe_filename="$(arg output_recipe_filename)" input_recipe_filename="$(arg input_recipe_filename)" reverse_ip="$(arg reverse_ip)" script_command_port="$(arg script_command_port)" reverse_port="$(arg reverse_port)" script_sender_port="$(arg script_sender_port)" trajectory_port="$(arg trajectory_port)">
+      <xacro:insert_block name="origin" />
+    </xacro:ur_robot>
+    <!-- Conditional inclusion for Gazebo simulation setup -->
+    <xacro:if value="$(arg sim_gazebo)">
+      <!-- Gazebo plugins -->
+      <gazebo reference="world">
+      </gazebo>
+      <gazebo>
+        <plugin filename="libgazebo_ros2_control.so" name="gazebo_ros2_control">
+          <parameters>$(arg simulation_controllers)</parameters>
+        </plugin>
+      </gazebo>
+    </xacro:if>
+    <xacro:if value="$(arg sim_ignition)">
+      <!-- Gazebo plugins -->
+      <gazebo reference="world">
+      </gazebo>
+      <gazebo>
+        <plugin filename="libign_ros2_control-system.so" name="ign_ros2_control::IgnitionROS2ControlPlugin">
+          <parameters>$(arg simulation_controllers)</parameters>
+          <controller_manager_node_name>$(arg tf_prefix)controller_manager</controller_manager_node_name>
+        </plugin>
+      </gazebo>
+    </xacro:if>
+  </xacro:macro>
 </robot>

File: hrwros_week3/hrwros_support/urdf/bin/bin.urdf.xacro (robot description, xacro)
@@ -1,5 +1,5 @@
 <?xml version="1.0"?>
 <robot xmlns:xacro="http://www.ros.org/wiki/xacro">
-  <xacro:macro name="bin_urdf" params="prefix *origin">
+  <xacro:macro name="bin_urdf" params="prefix bin_parent *origin">
     <!-- link list -->
     <link name="${prefix}base_link">
@@ -36,5 +36,10 @@
     </link>
     <!-- joint list -->
-    <joint name="${prefix}joint_2" type="fixed">
+    <joint name="${prefix}world_joint" type="fixed">
+      <xacro:insert_block name="origin" />
+      <parent link="${bin_parent}"/>
+      <child link="${prefix}base_link"/>
+    </joint>
+    <joint name="${prefix}joint_1" type="fixed">
       <origin xyz="0 0 1.0" rpy="0 0 0" />
       <parent link="${prefix}base_link" />

File: hrwros_week3/hrwros_support/urdf/bin/bin.xacro (robot description, xacro)
@@ -3,7 +3,9 @@
   xmlns:xacro="http://www.ros.org/wiki/xacro">
   <xacro:arg name="prefix" default="bin_1_"/>
+  <xacro:arg name="bin_parent" default="world_interface"/>
+  <link name="$(arg bin_parent)"/>
   <!-- URDF -->
   <xacro:include filename="$(find hrwros_support)/urdf/bin/bin.urdf.xacro"/>
-  <xacro:bin_urdf prefix="$(arg prefix)">
+  <xacro:bin_urdf prefix="$(arg prefix)" bin_parent="$(arg bin_parent)">
     <origin xyz="-8.0 -2.2 0.0" rpy="0 0 0" />
   </xacro:bin_urdf>

File: hrwros_week3/hrwros_support/urdf/break_beam/break_beam.urdf.xacro (robot description, xacro)
@@ -2,7 +2,6 @@
 <robot name="break_beam_urdf"
   xmlns:xacro="http://www.ros.org/wiki/xacro">
-  <xacro:macro name="break_beam_urdf" params="prefix *origin">
+  <xacro:macro name="break_beam_urdf" params="prefix break_beam_parent *origin">
     <!-- link list -->
-    <link name="${prefix}world_interface"/>
     <link name="${prefix}base_link">
       <visual>
@@ -31,5 +30,5 @@
     <!-- joint list -->
     <joint name="${prefix}world_joint" type="fixed">
-      <parent link="${prefix}world_interface" />
+      <parent link="${break_beam_parent}" />
       <child link="${prefix}base_link" />
       <xacro:insert_block name="origin" />

File: hrwros_week3/hrwros_support/urdf/break_beam/break_beam.xacro (robot description, xacro)
@@ -3,7 +3,9 @@
   xmlns:xacro="http://www.ros.org/wiki/xacro">
   <xacro:arg name="prefix" default="break_beam_"/>
+  <xacro:arg name="break_beam_parent" default="world_interface"/>
   <!-- URDF -->
+  <link name="$(arg break_beam_parent)"/>
   <xacro:include filename="$(find hrwros_support)/urdf/break_beam/break_beam.urdf.xacro"/>
-  <xacro:break_beam_urdf prefix="$(arg prefix)">
+  <xacro:break_beam_urdf prefix="$(arg prefix)" break_beam_parent="$(arg break_beam_parent)">
     <origin xyz="1.6 1.9 0.925" rpy="0 0 ${radians(180)}" />
   </xacro:break_beam_urdf>

File: hrwros_week3/hrwros_support/urdf/hrwros.xacro (robot description, xacro)
@@ -22,12 +22,12 @@
   <xacro:property name="vacuum_gripper2" value="vacuum_gripper2_"/>
   <!-- Workcell -->
-  <xacro:workcell_urdf workcell_parent_name="world_interface"/>
+  <xacro:workcell_urdf workcell_parent_name="world"/>
   <!-- Robots -->
   <!-- Robot1 Pedestal -->
-  <xacro:robot_pedestal_urdf pedestal_prefix="${robot1}_" pedestal_parent="world_interface" pedestal_height="${pedestal1_height}">
+  <xacro:robot_pedestal_urdf pedestal_prefix="${robot1}_" pedestal_parent="world" pedestal_height="${pedestal1_height}">
     <origin xyz="0.5 1.8 0.0" rpy="0 0 0"/>
   </xacro:robot_pedestal_urdf>
   <!-- Robot1 -->
-  <xacro:ur_description robot_name="${robot1}" ur_type="${ur_type1}">
+  <xacro:ur_description robot_name="${robot1}" ur_type="${ur_type1}" robot_parent="world">
     <origin xyz="0.5 1.8 ${pedestal1_height}" rpy="0 0 0"/>
   </xacro:ur_description>
@@ -35,9 +35,9 @@
   <xacro:vacuum_gripper_urdf prefix="${vacuum_gripper1}" />
   <!-- Robot2 Pedestal -->
-  <xacro:robot_pedestal_urdf pedestal_prefix="${robot2}_" pedestal_parent="world_interface" pedestal_height="${pedestal2_height}">
+  <xacro:robot_pedestal_urdf pedestal_prefix="${robot2}_" pedestal_parent="world" pedestal_height="${pedestal2_height}">
     <origin xyz="-7.8 -1.5 0.0" rpy="0 0 0"/>
   </xacro:robot_pedestal_urdf>
   <!-- Robot2 -->
-  <xacro:ur_description robot_name="${robot2}" ur_type="${ur_type2}">
+  <xacro:ur_description robot_name="${robot2}" ur_type="${ur_type2}" robot_parent="world">
     <origin xyz="-7.8 -1.5 ${pedestal2_height}" rpy="0 0 0"/>
   </xacro:ur_description>
@@ -46,25 +46,20 @@
   <!-- Bins -->
   <!-- Bin1 -->
-  <xacro:bin_urdf prefix="bin_1_">
+  <xacro:bin_urdf prefix="bin_1_" bin_parent="world">
     <origin xyz="-8.0 -2.2 0.0" rpy="0 0 0" />
   </xacro:bin_urdf>
   <!-- Logical Cameras -->
   <!-- Logical Camera 1 -->
-  <xacro:logical_camera_urdf prefix="logical_camera1_" logical_camera_parent="world_interface">
+  <xacro:logical_camera_urdf prefix="logical_camera1_" logical_camera_parent="world">
     <origin xyz="1.2 1.8 2.0" rpy="0 1.5708 0"/>
   </xacro:logical_camera_urdf>
   <!-- Logical Camera 2 -->
-  <xacro:logical_camera_urdf prefix="logical_camera2_" logical_camera_parent="world_interface">
+  <xacro:logical_camera_urdf prefix="logical_camera2_" logical_camera_parent="world">
     <origin xyz="-8.3 -1.23 1.8" rpy="0 1.5708 0"/>
   </xacro:logical_camera_urdf>
   <!-- Break Beam -->
-  <xacro:break_beam_urdf prefix="break_beam_">
+  <xacro:break_beam_urdf prefix="break_beam_" break_beam_parent="world">
     <origin xyz="1.6 1.9 0.925" rpy="0 0 ${radians(180)}" />
   </xacro:break_beam_urdf>
-  <!-- Joints -->
-  <joint name="world_interface_to_world" type="fixed">
-    <parent link="world" />
-    <child link="world_interface" />
-  </joint>
   <!-- gripper1 to robot1. -->
   <joint name="gripper1_to_robot1" type="fixed">
@@ -77,13 +72,3 @@
     <child link="${vacuum_gripper2}base_link" />
   </joint>
-  <joint name="bin_1_joint" type="fixed">
-    <parent link="world_interface" />
-    <child link="bin_1_base_link" />
-    <origin xyz="-8.0 -2.2 0.0" rpy="0 0 0" />
-  </joint>
-  <!-- break beam to world. -->
-  <joint name="break_beam_joint" type="fixed">
-    <parent link="world_interface" />
-    <child link="break_beam_world_interface" />
-  </joint>
 </robot>

File: hrwros_week3/hrwros_support/urdf/logical_camera/logical_camera.urdf.xacro (robot description, xacro)
@@ -6,5 +6,5 @@
     <xacro:property name="width" value="0.050"/>
     <xacro:property name="height" value="0.050"/>
-    <joint name="${prefix}logical_camera_joint" type="fixed">
+    <joint name="${prefix}world_joint" type="fixed">
       <xacro:insert_block name="origin" />
       <parent link="${logical_camera_parent}"/>

File: hrwros_week3/hrwros_support/urdf/logical_camera/logical_camera1.xacro (robot description, xacro)
@@ -3,6 +3,7 @@
   xmlns:xacro="http://www.ros.org/wiki/xacro">
   <xacro:arg name="prefix" default="logical_camera1_"/>
-  <link name="world_interface"/>
+  <xacro:arg name="logical_camera_parent" default="world_interface"/>
   <!-- URDF -->
+  <link name="$(arg logical_camera_parent)"/>
   <xacro:include filename="$(find hrwros_support)/urdf/logical_camera/logical_camera.urdf.xacro"/>
   <xacro:logical_camera_urdf prefix="$(arg prefix)" logical_camera_parent="$(arg logical_camera_parent)">

File: hrwros_week3/hrwros_support/urdf/logical_camera/logical_camera2.xacro (robot description, xacro)
@@ -4,6 +4,6 @@
   <xacro:arg name="prefix" default="logical_camera2_"/>
   <xacro:arg name="logical_camera_parent" default="world_interface"/>
-  <link name="world_interface"/>
   <!-- URDF -->
+  <link name="$(arg logical_camera_parent)"/>
   <xacro:include filename="$(find hrwros_support)/urdf/logical_camera/logical_camera.urdf.xacro"/>
   <xacro:logical_camera_urdf prefix="$(arg prefix)" logical_camera_parent="$(arg logical_camera_parent)">

File: hrwros_week3/hrwros_support/urdf/robot_pedestal/robot1_pedestal.xacro (robot description, xacro)
@@ -1,8 +1,9 @@
 <?xml version="1.0" ?>
-<robot name="robot_pedestal" xmlns:xacro="http://www.ros.org/wiki/xacro">
+<robot name="robot_pedestal"
+  xmlns:xacro="http://www.ros.org/wiki/xacro">
   <xacro:arg name="pedestal_prefix" default="robot1"/>
   <xacro:arg name="pedestal_parent" default="world_interface"/>
   <xacro:arg name="pedestal_height" default="0.95"/>
-  <link name="world_interface"/>
+  <link name="$(arg pedestal_parent)"/>
   <!-- URDF -->
   <xacro:include filename="$(find hrwros_support)/urdf/robot_pedestal/robot_pedestal.urdf.xacro"/>

File: hrwros_week3/hrwros_support/urdf/robot_pedestal/robot2_pedestal.xacro (robot description, xacro)
@@ -5,5 +5,5 @@
   <xacro:arg name="pedestal_parent" default="world_interface"/>
   <xacro:arg name="pedestal_height" default="0.5"/>
-  <link name="world_interface"/>
+  <link name="$(arg pedestal_parent)"/>
   <!-- URDF -->
   <xacro:include filename="$(find hrwros_support)/urdf/robot_pedestal/robot_pedestal.urdf.xacro"/>

File: hrwros_week3/hrwros_support/urdf/robot_pedestal/robot_pedestal.urdf.xacro (robot description, xacro)
@@ -25,5 +25,5 @@
     </inertial>
   </link>
-  <joint name="${pedestal_prefix}pedestal_joint" type="fixed">
+  <joint name="${pedestal_prefix}world_joint" type="fixed">
     <xacro:insert_block name="origin" />
     <parent link="${pedestal_parent}"/>

File: hrwros_week3/hrwros_support/urdf/robot_system/robot_system.urdf.xacro (robot description, xacro)
@@ -2,12 +2,12 @@
 <robot name="robot_system"
   xmlns:xacro="http://www.ros.org/wiki/xacro">
-  <xacro:macro name="robot_system_urdf" params="robot_prefix vacuum_gripper_prefix robot_type">
+  <xacro:macro name="robot_system_urdf" params="robot_prefix vacuum_gripper_prefix robot_type robot_parent">
     <xacro:arg name="transmission_hw_interface" default="hardware_interface/EffortJointInterface" />
     <xacro:include filename="$(find hrwros_support)/urdf/arm_robot/ur_description.urdf.xacro"/>
     <xacro:include filename="$(find hrwros_support)/urdf/vacuum_gripper/vacuum_gripper.urdf.xacro"/>
     <!-- Used for fixing robot to Gazebo 'base_link' -->
-    <link name="world_interface"/>
+    <link name="${robot_parent}"/>
     <!-- Robot1 -->
-    <xacro:ur_description robot_name="${robot_prefix}" ur_type="${robot_type}">
+    <xacro:ur_description robot_name="${robot_prefix}" ur_type="${robot_type}" robot_parent="${robot_parent}">
       <!-- <origin xyz="0.0 0.0 ${pedestal1_height}" rpy="0 0 0"/> -->
       <origin xyz="0.0 0.0 0.0" rpy="0 0 0"/>

File: hrwros_week3/hrwros_support/urdf/robot_system/robot_system.xacro (robot description, xacro)
@@ -7,7 +7,8 @@
   <xacro:arg name="robot_param" default=""/>
   <xacro:arg name="gripper_plugin_name" default="gripper1"/>
+  <xacro:arg name="robot_parent" default="world_interface"/>
   <!-- URDF -->
   <xacro:include filename="$(find hrwros_support)/urdf/robot_system/robot_system.urdf.xacro"/>
-  <xacro:robot_system_urdf robot_type= "$(arg robot_type)" robot_prefix="$(arg robot_prefix)" vacuum_gripper_prefix="$(arg vacuum_gripper_prefix)"/>
+  <xacro:robot_system_urdf robot_type= "$(arg robot_type)" robot_prefix="$(arg robot_prefix)" vacuum_gripper_prefix="$(arg vacuum_gripper_prefix)" robot_parent="$(robot_parent)"/>
   <!-- Gazebo -->
   <xacro:include filename="$(find hrwros_support)/urdf/robot_system/robot_system.gazebo.xacro"/>

File: hrwros_week3/hrwros_support/urdf/workcell/workcell.urdf.xacro (robot description, xacro)
@@ -3,5 +3,4 @@
     <xacro:macro name="workcell_urdf" params="workcell_parent_name">
     <!-- Links -->
-    <link name="world_interface"/>
     <link name="workcell">
       <visual>

File: hrwros_week3/hrwros_support/urdf/workcell/workcell.xacro (robot description, xacro)
@@ -4,4 +4,5 @@
   <xacro:arg name="workcell_parent_name" default="world_interface"/>
   <!-- URDF -->
+  <link name="$(arg workcell_parent_name)"/>
   <xacro:include filename="$(find hrwros_support)/urdf/workcell/workcell.urdf.xacro"/>
   <xacro:workcell_urdf workcell_parent_name="$(arg workcell_parent_name)"/>
