Commit message: fix controller manager and namespace

File: hrwros_week3/hrwros_support/urdf/arm_robot/arm_description.urdf.xacro (robot description, xacro)
@@ -26,4 +26,5 @@
       <gazebo>
         <plugin filename="libgazebo_ros2_control.so" name="gazebo_ros2_control">
+          <namespace>${robot_name}</namespace>
           <parameters>$(arg simulation_controllers)</parameters>
         </plugin>

File: hrwros_week3/hrwros_support/urdf/robot_system/robot_system.gazebo.xacro (robot description, xacro)
@@ -2,5 +2,5 @@
 <robot name="robot_system"
   xmlns:xacro="http://www.ros.org/wiki/xacro">
-  <xacro:macro name="robot_system_gazebo" params="robot_prefix robot_parameter_name vacuum_gripper_prefix gripper_plugin_name">
+  <xacro:macro name="robot_system_gazebo" params="robot_prefix vacuum_gripper_prefix gripper_plugin_name">
     <!-- Vacuum Gripper -->
     <xacro:if value="${robot_prefix == 'robot1_'}">

File: hrwros_week3/hrwros_support/urdf/robot_system/robot_system.xacro (robot description, xacro)
@@ -5,5 +5,4 @@
   <xacro:arg name="robot_prefix" default="robot1"/>
   <xacro:arg name="vacuum_gripper_prefix" default="vacuum_gripper1_"/>
-  <xacro:arg name="robot_param" default=""/>
   <xacro:arg name="gripper_plugin_name" default="gripper1"/>
   <xacro:arg name="robot_parent" default="world_interface"/>
@@ -13,4 +12,4 @@
   <!-- Gazebo -->
   <xacro:include filename="$(find hrwros_support)/urdf/robot_system/robot_system.gazebo.xacro"/>
-  <xacro:robot_system_gazebo robot_prefix="$(arg robot_prefix)" robot_parameter_name="$(arg robot_param)" vacuum_gripper_prefix="$(arg vacuum_gripper_prefix)" gripper_plugin_name="$(arg gripper_plugin_name)"/>
+  <xacro:robot_system_gazebo robot_prefix="$(arg robot_prefix)" vacuum_gripper_prefix="$(arg vacuum_gripper_prefix)" gripper_plugin_name="$(arg gripper_plugin_name)"/>
 </robot>
