Commit message: small change in turtlebot publisher

File: hrwros_week3/hrwros_support/urdf/mobile_robot/mobile_robot.urdf.xacro (robot description, xacro)
@@ -5,11 +5,11 @@
     <xacro:include filename="$(find turtlebot3_gazebo)/urdf/turtlebot3_${turtlebot_model}.urdf"/>
     <!-- Used for fixing robot to Gazebo 'base_footprint' -->
-    <link name="${robot_parent}"/>
+    <!-- <link name="${robot_parent}"/> -->
     <!-- turtlebotto to world. -->
-    <joint name="${turtlebot_model}_turtlebot_world_joint" type="fixed">
+    <!-- <joint name="${turtlebot_model}_turtlebot_world_joint" type="fixed">
       <xacro:insert_block name="origin" />
       <parent link="${robot_parent}" />
       <child link="base_footprint" />
-    </joint>
+    </joint> -->
   </xacro:macro>
 </robot>
